Commit message: Plugin can move joints with position controller

File: ros2_description_solo12/ros2_control/system_solo12.ros2_control.xacro (robot description, xacro)
@@ -6,6 +6,6 @@
         <hardware>
           <plugin>gazebo_ros2_control_bolt/GazeboBoltSystem</plugin>
-	  <param name="default_kp">1000.0</param>
-	  <param name="default_kd">10.0</param>
+          <param name="default_kp">1000.0</param>
+          <param name="default_kd">10.0</param>
         </hardware>
       </xacro:if>
@@ -13,31 +13,5 @@
         <hardware>
           <xacro:if value="${use_fake_hardware}">
-            <plugin>fake_components/GenericSystem</plugin><joint name="FL_HFE">
-        <command_interface name="position">
-          <param name="min">-1.45</param>
-          <param name="max">1.45</param>
-        </command_interface>
-        <command_interface name="velocity">
-          <param name="min">-1</param>
-          <param name="max">1</param>
-        </command_interface>
-        <command_interface name="effort">
-          <param name="min">-1</param>
-          <param name="max">1</param>
-        </command_interface>
-        <command_interface name="gain_kp">
-          <param name="min">-1000</param>
-          <param name="max">1000</param>
-        </command_interface>
-        <command_interface name="gain_kd">
-          <param name="min">-1000</param>
-          <param name="max">1000</param>
-        </command_interface>
-        <state_interface name="position"/>
-        <state_interface name="velocity"/>
-        <state_interface name="effort"/>
-        <state_interface name="gain_kp"/>
-        <state_interface name="gain_kd"/>
-      </joint>
+            <plugin>fake_components/GenericSystem</plugin>
             <param name="fake_sensor_commands">${fake_sensor_commands}</param>
             <param name="state_following_offset">0.0</param>
@@ -110,5 +84,5 @@
         <state_interface name="gain_kd"/>
       </joint>
-      <joint name="FL_K">
+      <joint name="FL_KFE">
         <command_interface name="position">
           <param name="min">-2.8</param>
@@ -191,5 +165,5 @@
         <state_interface name="gain_kd"/>
       </joint>
-      <joint name="FR_K">
+      <joint name="FR_KFE">
         <command_interface name="position">
           <param name="min">-2.8</param>
@@ -272,5 +246,5 @@
         <state_interface name="gain_kd"/>
       </joint>
-      <joint name="HL_K">
+      <joint name="HL_KFE">
         <command_interface name="position">
           <param name="min">-2.8</param>
@@ -353,5 +327,5 @@
         <state_interface name="gain_kd"/>
       </joint>
-      <joint name="HR_K">
+      <joint name="HR_KFE">
         <command_interface name="position">
           <param name="min">-2.8</param>

File: ros2_description_solo12/urdf/system_solo12.urdf.xacro (robot description, xacro)
@@ -89,4 +89,4 @@
       color="${color}"
       opacity="${opacity}"/>
-  </xacro:macro>
+</xacro:macro>
 </robot>

File: ros2_description_solo12/urdf/system_solo12_description.urdf.xacro (robot description, xacro)
@@ -27,7 +27,14 @@
     </xacro:if>
   </xacro:if>
-  <!-- <xacro:include filename="$(find ros2_description_solo12)/ros2_control/system_solo12.ros2_control.xacro" /> -->
+  <xacro:include filename="$(find ros2_description_solo12)/ros2_control/system_solo12.ros2_control.xacro" />
   <!-- ros_control plugin for Gazebo -->
   <!-- THE PLUGIN IS MISSING -->
+  <xacro:if value="$(arg use_sim)">
+    <gazebo>
+      <plugin name="gazebo_ros2_bolt" filename="libgazebo_ros2_control_solo12.so">
+	    <parameters>$(find gazebo_ros2_control_solo12)/config/bolt_gazebo_config_controller.yaml</parameters>
+      </plugin>
+    </gazebo>
+  </xacro:if>
   <xacro:if value="$(arg use_sim)">
     <xacro:if value="$(arg use_crane)">
@@ -42,6 +49,6 @@
       opacity="${opacity}"
         />
-  <!-- <xacro:system_solo112_ros2_control
+  <xacro:system_solo12_ros2_control
     name="SystemBoltRos2Control" prefix="$(arg prefix)" use_fake_hardware="$(arg use_fake_hardware)"
-      use_sim="$(arg use_sim)"/> -->
+      use_sim="$(arg use_sim)"/>
 </robot>
